File: esquemático.brd (EAGLE design)
At the start: 70.1 x 59.1 mm, 28 parts, among them Q1 MMBT4403LT1SMD, Q3 MMBT4403LT1SMD, X1 MKDSN1,5/2-5,08, X2 MKDSN1,5/2-5,08, X3 MKDSN1,5/2-5,08, X4 MKDSN1,5/2-5,08

Commit message: Add files via upload
Parts:
- renumbered ADC1 to U1, ADC2 to U2, LDO to U3
Changed lines of the file:
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@@
 </autorouter>
 <elements>
-<element name="ADC1" library="HX711" package="SOIC127P600X140-16N" package3d_urn="urn:adsk.eagle:package:38132012/1" value="" x="50.8" y="29.464" smashed="yes">
+<element name="U1" library="HX711" package="SOIC127P600X140-16N" package3d_urn="urn:adsk.eagle:package:38132012/1" value="" x="50.8" y="29.464" smashed="yes">
 <attribute name="NAME" x="50.8" y="35.0868" size="1.016" layer="25" align="bottom-center"/>
 <attribute name="VALUE" x="50.8" y="23.779" size="1.27" layer="27" align="top-center"/>
 </element>
-<element name="ADC2" library="HX711" package="SOIC127P600X140-16N" package3d_urn="urn:adsk.eagle:package:38132012/1" value="" x="29.972" y="29.718" smashed="yes">
+<element name="U2" library="HX711" package="SOIC127P600X140-16N" package3d_urn="urn:adsk.eagle:package:38132012/1" value="" x="29.972" y="29.718" smashed="yes">
 <attribute name="NAME" x="29.972" y="35.3408" size="1.016" layer="25" align="bottom-center"/>
 <attribute name="VALUE" x="29.972" y="24.033" size="1.27" layer="27" align="top-center"/>
@@
 <attribute name="VALUE" x="29.8958" y="3.3528" size="1.27" layer="27" rot="R90"/>
 </element>
-<element name="LDO" library="Celda_Carga" package="SOT-23-3" value="AP2210N-4.0TRG1" x="18.288" y="46.99" smashed="yes" rot="R90">
+<element name="U3" library="Celda_Carga" package="SOT-23-3" value="AP2210N-4.0TRG1" x="18.288" y="46.99" smashed="yes" rot="R90">
 <attribute name="NAME" x="16.012" y="47.276" size="1.016" layer="25" rot="R180"/>
 </element>
@@
 <contactref element="M1" pad="CN10-9"/>
 <contactref element="M1" pad="CN10-20"/>
-<contactref element="ADC1" pad="14"/>
-<contactref element="ADC1" pad="10"/>
-<contactref element="ADC1" pad="9"/>
+<contactref element="U1" pad="14"/>
+<contactref element="U1" pad="10"/>
+<contactref element="U1" pad="9"/>
 <contactref element="C1" pad="2"/>
 <contactref element="X1" pad="1"/>
 <contactref element="R2" pad="2"/>
-<contactref element="ADC1" pad="5"/>
+<contactref element="U1" pad="5"/>
 <contactref element="C3" pad="1"/>
 <contactref element="C2" pad="2"/>
-<contactref element="LDO" pad="1"/>
+<contactref element="U3" pad="1"/>
 <contactref element="C5" pad="2"/>
 <contactref element="C6" pad="2"/>
-<contactref element="ADC2" pad="14"/>
-<contactref element="ADC2" pad="10"/>
-<contactref element="ADC2" pad="9"/>
+<contactref element="U2" pad="14"/>
+<contactref element="U2" pad="10"/>
+<contactref element="U2" pad="9"/>
 <contactref element="C7" pad="2"/>
 <contactref element="X4" pad="1"/>
 <contactref element="R6" pad="2"/>
-<contactref element="ADC2" pad="5"/>
+<contactref element="U2" pad="5"/>
 <contactref element="C9" pad="1"/>
 <contactref element="C8" pad="2"/>
@@
 </signal>
 <signal name="N$1">
-<contactref element="ADC1" pad="3"/>
+<contactref element="U1" pad="3"/>
 <contactref element="X1" pad="2"/>
 <contactref element="R1" pad="1"/>
@@
 <signal name="N$4">
 <contactref element="R2" pad="1"/>
-<contactref element="ADC1" pad="4"/>
+<contactref element="U1" pad="4"/>
 <contactref element="R1" pad="2"/>
 <wire x1="48.0967" y1="30.099" x2="47.437" y2="30.099" width="0.254" layer="1"/>
@@
 </signal>
 <signal name="N$2">
-<contactref element="ADC1" pad="7"/>
+<contactref element="U1" pad="7"/>
 <contactref element="R3" pad="2"/>
 <contactref element="C4" pad="1"/>
@@
 </signal>
 <signal name="N$6">
-<contactref element="ADC1" pad="8"/>
+<contactref element="U1" pad="8"/>
 <contactref element="R4" pad="2"/>
 <contactref element="C4" pad="2"/>
@@
 </signal>
 <signal name="N$8">
-<contactref element="ADC1" pad="6"/>
+<contactref element="U1" pad="6"/>
 <contactref element="C3" pad="2"/>
 <wire x1="48.0967" y1="27.559" x2="45.659" y2="27.559" width="0.254" layer="1"/>
@@
 </signal>
 <signal name="VCC">
-<contactref element="LDO" pad="3"/>
+<contactref element="U3" pad="3"/>
 <contactref element="C5" pad="1"/>
 <contactref element="M1" pad="CN6-5"/>
@@
 </signal>
 <signal name="N$10">
-<contactref element="ADC1" pad="2"/>
+<contactref element="U1" pad="2"/>
 <contactref element="Q3" pad="B"/>
 <wire x1="48.0967" y1="32.639" x2="47.371" y2="32.639" width="0.254" layer="1"/>
@@
 </signal>
 <signal name="N$9">
-<contactref element="ADC2" pad="3"/>
+<contactref element="U2" pad="3"/>
 <contactref element="X4" pad="2"/>
 <contactref element="R5" pad="1"/>
@@
 <signal name="N$11">
 <contactref element="R6" pad="1"/>
-<contactref element="ADC2" pad="4"/>
+<contactref element="U2" pad="4"/>
 <contactref element="R5" pad="2"/>
 <wire x1="27.2687" y1="30.353" x2="26.57485" y2="31.04685" width="0.254" layer="1"/>
@@
 </signal>
 <signal name="N$12">
-<contactref element="ADC2" pad="7"/>
+<contactref element="U2" pad="7"/>
 <contactref element="R7" pad="2"/>
 <contactref element="C10" pad="1"/>
@@
 </signal>
 <signal name="N$14">
-<contactref element="ADC2" pad="8"/>
+<contactref element="U2" pad="8"/>
 <contactref element="R8" pad="2"/>
 <contactref element="C10" pad="2"/>
@@
 </signal>
 <signal name="N$16">
-<contactref element="ADC2" pad="6"/>
+<contactref element="U2" pad="6"/>
 <contactref element="C9" pad="2"/>
 <wire x1="27.2687" y1="27.813" x2="26.035" y2="27.813" width="0.254" layer="1"/>
@@
 </signal>
 <signal name="N$18">
-<contactref element="ADC2" pad="2"/>
+<contactref element="U2" pad="2"/>
 <contactref element="Q1" pad="B"/>
 <wire x1="27.2687" y1="32.893" x2="27.1417" y2="32.766" width="0.254" layer="1"/>
@@
 <signal name="N$3">
 <contactref element="M1" pad="CN9-8"/>
-<contactref element="ADC1" pad="11"/>
-<contactref element="ADC2" pad="11"/>
+<contactref element="U1" pad="11"/>
+<contactref element="U2" pad="11"/>
 <wire x1="59.13" y1="22.852" x2="56.896" y2="22.852" width="0.254" layer="1"/>
 <wire x1="56.896" y1="22.852" x2="48.506" y2="22.852" width="0.254" layer="1"/>
@@
 </signal>
 <signal name="N$19">
-<contactref element="ADC1" pad="12"/>
+<contactref element="U1" pad="12"/>
 <contactref element="M1" pad="CN8-5"/>
 <wire x1="10.87" y1="7.612" x2="13.708" y2="7.612" width="0.254" layer="1"/>
@@
 <signal name="N$20">
 <contactref element="M1" pad="CN8-6"/>
-<contactref element="ADC2" pad="12"/>
+<contactref element="U2" pad="12"/>
 <wire x1="10.87" y1="5.072" x2="10.878" y2="5.08" width="0.254" layer="1"/>
 <wire x1="10.878" y1="5.08" x2="14.732" y2="5.08" width="0.254" layer="1"/>
@@
 </signal>
 <signal name="N$22">
-<contactref element="ADC2" pad="15"/>
-<contactref element="ADC1" pad="15"/>
+<contactref element="U2" pad="15"/>
+<contactref element="U1" pad="15"/>
 <contactref element="C7" pad="1"/>
-<contactref element="ADC2" pad="1"/>
-<contactref element="ADC2" pad="16"/>
+<contactref element="U2" pad="1"/>
+<contactref element="U2" pad="16"/>
 <contactref element="C1" pad="1"/>
-<contactref element="ADC1" pad="1"/>
-<contactref element="ADC1" pad="16"/>
-<contactref element="LDO" pad="2"/>
+<contactref element="U1" pad="1"/>
+<contactref element="U1" pad="16"/>
+<contactref element="U3" pad="2"/>
 <contactref element="C6" pad="1"/>
 <contactref element="Q3" pad="E"/>
