File: esquemático.sch (EAGLE design)
At the start: 28 parts, among them Q1 MMBT4403LT1SMD, Q3 MMBT4403LT1SMD, X1 MKDSN1,5/2-5,08, X2 MKDSN1,5/2-5,08, X3 MKDSN1,5/2-5,08, X4 MKDSN1,5/2-5,08

Commit message: Add files via upload
Parts:
- renumbered ADC1 to U1, ADC2 to U2, LDO to U3

Commit message: Add files via upload
Parts:
- Q1, Q3: PARTNO (none) -> BCR573E6327
- U1, U2: PARTNO (none) -> HX711
- U3: PARTNO (none) -> AP2210N-4.0TRG1
- X1, X2, X3, X4: PARTNO (none) -> MKDSN1,5/2-5,08
